Commit message: keys go in: the insertion trains once the key can tilt in the hand and the task layer closes its loops on the measured tip, 80-83 of 96 in PhysX; the D1 measured onto the EDU's dock, and the dock drawn
- Insertion (demos/insertion, unifp_train/insertion*, insert_*): a keyed-slot plant, a force-law task layer with a
  spiral search and a home hold, outer loops on the key's tip, the approach's elevation and the blade's roll, and a
  compliant grip (analytic, and in PhysX as two sprung joints on the key). Trained v5-v11 and three seeds; the best
  checkpoints seat 71-75/96 frozen 1 mm slots and 80-83/96 in PhysX at a 2 mm estimate error, no damage, no falls
  (checkpoints/unifp_go2d1_insertion_seed3_model_21200.pt, ..._model_21400.pt). F-116, F-119-F-122.
- The D1's mount measured off Unitree's Go2-with-dock CAD and applied everywhere from mount.py (F-117); how much the
  reaching policy depends on it (F-118); the expansion dock and rails drawn in the sim, RViz and the cup console
  (dock.py, description/dock_from_cad.py, third_party/unitree_go2_cad).
- The mechanism policy trained on levers and high handles (F-114, F-115; checkpoints/..._mech_lever_model_20497.pt).
- Launcher: loop gains and clamps, the compliant grip, the home hold, the curriculum's pace, the arm's action noise
  on resume; the insertion demo runs in batches; run_camera_body_view renders the dock and starts again.
- Week 2 log and findings, with every run recorded.

Co-Authored-By: Claude Opus 5.5 (1M context) <noreply@anthropic.com>

File: description/go2_d1.urdf (robot description, URDF)
Before this commit: robot go2_d1, 39 links, 38 joints
Links:
- added link expansion_dock; visual mesh filename=package://d1_training/description/meshes/go2/expansion_dock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; visual mesh filename=package://d1_training/description/meshes/go2/expansion_dock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
Joints:
- added joint expansion_dock_joint: type fixed, parent base_link, child expansion_dock, origin xyz=0 0 0 rpy=0 0 0
- joint arm_mount_joint: origin xyz=0 0 0.08 rpy=0 0 0 -> xyz=0.0025 0 0.0855 rpy=0 0 0

Commit message: Put the D1 where it really sits: on the rails' screw positions and on its measured base (F-078, F-079)
Lukas measured the real arm. Its holes are 13 cm apart along the rail, matching the Go2 EDU
rails' own screws (131.0 mm apart in Unitree's rail CAD, x = -84.5 and +46.6 mm, rail tops
at z = 85.5 mm). Its base is one 126 mm cylinder, 76 mm from its bottom to the rotating
plate. Unitree's base_link.STL is 105 mm and 53.3 mm, 1.20x in plan and 1.43x in height,
so it is a different part. Above the plate the model is right: the shoulder height checks,
and the chain reaches 554.9 mm against the published 550.

- weld.D1_MOUNT_POS = (-0.019, 0, 0.0855) is the one mount, replacing (0, 0, 0.08).
  sim.py, run_position_only.py and the three demo launchers take it from there, and the
  CPU copies (workspace.MOUNT_B, the URDF builder) match it. run.json records arm_mount_m.
  sim.py's teleop reach clamp measures from the mount's x too.
- d1_arm/measured_base.py writes base_link_measured.STL: Unitree's base scaled 1.20 in plan
  with the cylinder stretched to 76 mm. d1.urdf uses it, carries the base's centre of mass
  and puts Joint1 at 76.0 mm. Unitree's mesh is kept. go2_d1.urdf's mount joint, Joint1 and
  base mesh were edited in place (a regeneration now pulls in P2Dingo's newer links; see
  description/README.md), and d1_ui's shoulder height was updated.
- Stance re-measured with the Week 1 probe, which reproduced the committed values exactly
  at the old mount as a control. Base (-0.0571, 0, 0.2736) m; resting tip
  (0.3378, -0.0141, 0.7906) m, into task_space. verify 25/25 at both steps, and the box is
  98.99% reachable. The frozen manifests are unchanged.
- Tests: the workspace pins moved with the arm. The level-IK point moved up with the
  shoulder: the arm now stops 22.5 mm short of the old one, a real loss of low level
  reach. Four demo tests still fail (pick survey, pivot, wide-cup grasp, combiner tag pose).
  Their scenes sit at fixed spots in the base frame, tuned for the old arm, and are left
  for a decision (Week 3 notes).
- results/: Week 3 log entries, the two verify runs, probe and workspace evidence, the
  photograph of the base; F-078 (mount, superseded for its stance numbers) and F-079.

Co-Authored-By: Claude Opus 5.5 <noreply@anthropic.com>

File: description/go2_d1.urdf (robot description, URDF)
Before this commit: robot go2_d1, 39 links, 38 joints
Links:
- link d1_base_link: geometry collision mesh filename=package://d1_training/d1_arm/meshes/base_link_measured.STL; visual mesh filename=package://d1_training/d1_arm/meshes/base_link_measured.STL
Joints:
- joint Joint1: origin xyz=0 0 0.0533 rpy=0 0 -3.1416 -> xyz=0 0 0.076 rpy=0 0 -3.1416
- joint arm_mount_joint: origin xyz=0 0 0.08 rpy=0 0 0 -> xyz=-0.019 0 0.0855 rpy=0 0 0
