Commit message: Apply Unitree's published D1-550 spec; fix Joint3's effort limit
Lukas supplied the real spec from Unitree's D1 developer docs
(support.unitree.com/home/en/developer/D1Arm_services):

  Weight 3152 g | arm length 550 mm | rated load 500 g
  Torque  J0 3.3, J1 3.3, J2 1.7, J3 1.7, J4 1.7, J5 1.7, J6 1.7 Nm
  Range   J0 +/-135, J1 +/-90, J2 +/-90, J3 +/-135, J4 +/-90, J5 +/-135

This retracts the previous commit's claim that 3.33 Nm was "provably too
weak". It was not: that was an inference from a static-torque estimate,
asserted as proof. Unitree publishes 3.3 Nm and the URDF was right.

Mapping the spec onto the URDF (protocol J(N-1) -> URDF JointN, per
d1_protocol.py) does turn up one genuine error. All six ranges match
exactly, which confirms the offset -- but Joint3 carried 3.33 Nm where
J2 is rated 1.7. Whoever filled in the limits assumed "first three strong,
last three weak"; the D1 is first two strong, last four weak. Joint3 was
~2x too strong. Efforts are now 3.3/3.3/1.7/1.7/1.7/1.7 exactly.

Also decouples effort from mass. --arm_mass previously scaled the effort
limits alongside the mass, which was a workaround for not knowing the real
torques: it invented an arm whose motors grew with its weight. Unitree
publishes mass and per-joint torque as independent facts, so mass scaling
now touches mass and inertia only, and the drive gains no longer scale
either. arm_gain_scale is gone.

--arm_mass now defaults to 3.152, the published figure, so the sim is
right by default; pass 0.719 to get the URDF's own shells back. Confirmed
against Unitree's own d1_description: it ships the same 0.719 kg shell
inertials AND effort limits of zero, so there are no better numbers to be
had -- the hand-filled values were unavoidable.

At the published spec the dog still walks, but the arm droops:

  3.152 kg, 3.3/1.7 Nm   18.17 kg total   9.16 m   10.0 deg   stayed up
                                          arm EE error 31.5 cm

The droop is very likely an artefact of the uniform mass scaling rather
than a real D1 limitation: the missing 2.4 kg is servos sitting at the
joints, and smearing it evenly over the links loads the far end and
inflates the shoulder torque past its 3.3 Nm. Flagged in _rescale_arm's
docstring from the start; now demonstrably biting. Left as-is pending a
decision on whether to model the servo masses.

Co-Authored-By: Claude Opus 4.8 (1M context) <noreply@anthropic.com>

File: d1_arm/d1.urdf (robot description, URDF)
Before this commit: robot d1_description, 9 links, 8 joints
Joints:
- joint Joint1: limit lower=-2.35 upper=2.35 effort=3.33 velocity=1.05 -> lower=-2.35 upper=2.35 effort=3.3 velocity=1.05
- joint Joint2: limit lower=-1.57 upper=1.57 effort=3.33 velocity=1.05 -> lower=-1.57 upper=1.57 effort=3.3 velocity=1.05
- joint Joint3: limit lower=-1.57 upper=1.57 effort=3.33 velocity=1.05 -> lower=-1.57 upper=1.57 effort=1.7 velocity=1.05
- joint Joint4: limit lower=-2.35 upper=2.35 effort=1.67 velocity=1.73 -> lower=-2.35 upper=2.35 effort=1.7 velocity=1.73
- joint Joint5: limit lower=-1.57 upper=1.57 effort=1.67 velocity=1.73 -> lower=-1.57 upper=1.57 effort=1.7 velocity=1.73
- joint Joint6: limit lower=-2.35 upper=2.35 effort=1.67 velocity=1.73 -> lower=-2.35 upper=2.35 effort=1.7 velocity=1.73

Commit message: the D1 given Unitree's CAD lengths and a 3.33 N·m shoulder and elbow (F-139, F-140), the reach and rope policies retrained for it (F-141), and everything that reads the arm re-run
d1.urdf's five joint origins now follow Unitree's D1-550 CAD: the controlled point moves a median 6 mm,
the policies in use move by at most 4 episodes on their frozen sets, G0 passes 25/25. With Joint2 and
Joint3 at 3.33 N·m the old policies over-pull; the retrained rope policy holds 30 and 45 N with no fall
in 192 held-out releases by pulling with the arm. New checkpoints: unifp_go2d1_isaaclab_cad333_model_58400.pt
and unifp_go2d1_rope_cad333_model_14600.pt.

Written as F-138 to F-140 and renumbered F-139 to F-141 on merging origin/main (81b3a13), whose F-138
(the wrist camera's bracket) took the number first.

Co-Authored-By: Claude Opus 5.5 (1M context) <noreply@anthropic.com>

File: d1_arm/d1.urdf (robot description, URDF)
Before this commit: robot d1_description, 9 links, 8 joints
Joints:
- joint Joint2: limit lower=-1.57 upper=1.57 effort=3.3 velocity=1.05 -> lower=-1.57 upper=1.57 effort=3.33 velocity=1.05; origin xyz=0 0.028 0.0563 rpy=1.5708 0 -3.1416 -> xyz=0 0.028 0.0548 rpy=1.5708 0 -3.1416
- joint Joint3: limit lower=-1.57 upper=1.57 effort=1.7 velocity=1.05 -> lower=-1.57 upper=1.57 effort=3.33 velocity=1.05; origin xyz=0 0.2693 0.0009 rpy=0 0 0 -> xyz=0 0.27 0 rpy=0 0 0
- joint Joint4: origin xyz=0.0577 0.042 -0.0275 rpy=-1.5708 0 -1.5708 -> xyz=0.0577 0.041325 -0.0275 rpy=-1.5708 0 -1.5708
- joint Joint5: origin xyz=-0.0001 -0.0237 0.14018 rpy=1.5708 -1.5708 0 -> xyz=-0.0001 -0.0237 0.146973 rpy=1.5708 -1.5708 0
- joint Joint6: origin xyz=0.0825 -0.0010782 -0.023822 rpy=-1.5708 0 -1.5708 -> xyz=0.080781 -0.0010782 -0.023822 rpy=-1.5708 0 -1.5708

File: description/go2_d1.urdf (robot description, URDF)
Before this commit: robot go2_d1, 40 links, 39 joints
Joints:
- joint Joint2: limit lower=-1.57 upper=1.57 effort=3.3 velocity=1.05 -> lower=-1.57 upper=1.57 effort=3.33 velocity=1.05; origin xyz=0 0.028 0.0563 rpy=1.5708 0 -3.1416 -> xyz=0 0.028 0.0548 rpy=1.5708 0 -3.1416
- joint Joint3: limit lower=-1.57 upper=1.57 effort=1.7 velocity=1.05 -> lower=-1.57 upper=1.57 effort=3.33 velocity=1.05; origin xyz=0 0.2693 0.0009 rpy=0 0 0 -> xyz=0 0.27 0 rpy=0 0 0
- joint Joint4: origin xyz=0.0577 0.042 -0.0275 rpy=-1.5708 0 -1.5708 -> xyz=0.0577 0.041325 -0.0275 rpy=-1.5708 0 -1.5708
- joint Joint5: origin xyz=-0.0001 -0.0237 0.14018 rpy=1.5708 -1.5708 0 -> xyz=-0.0001 -0.0237 0.146973 rpy=1.5708 -1.5708 0
- joint Joint6: origin xyz=0.0825 -0.0010782 -0.023822 rpy=-1.5708 0 -1.5708 -> xyz=0.080781 -0.0010782 -0.023822 rpy=-1.5708 0 -1.5708
